File: Main Board - NDT.kicad_sch (KiCad schematic)
At the start: 0 parts

Commit message: finished, just produce fabrication outputs
Other:
- sheet MCU ports: added RF_RX_TX; removed none
- sheet RF ports: added RF_RX_TX; removed none
Changed lines of the file:
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@@
+	(wire
+		(pts
+			(xy 152.4 105.41) (xy 177.8 105.41)
+		)
+		(stroke
+			(width 0)
+			(type default)
+		)
+	)
 	(wire
 		(pts
@@
 	(sheet
 		(at 177.8 76.2)
-		(size 25.4 25.4)
+		(size 25.4 31.75)
 		(exclude_from_sim no)
 		(in_bom yes)
@@
 		)
 		(property "Sheetfile" "RF.kicad_sch"
-			(at 177.8 102.1846 0)
+			(at 177.8 108.5346 0)
 			(effects
 				(font
@@
 		(pin "RF_PA_P" bidirectional
 			(at 177.8 87.63 180)
+			(effects
+				(font
+					(size 1.27 1.27)
+				)
+				(justify left)
+			)
+		)
+		(pin "RF_RX_TX" input
+			(at 177.8 105.41 180)
 			(effects
 				(font
@@
 			)
 		)
+		(pin "RF_RX_TX" output
+			(at 152.4 105.41 0)
+			(effects
+				(font
+					(size 1.27 1.27)
+				)
+				(justify right)
+			)
+		)
