File: Main Board - NDT.kicad_pcb (KiCad board)
At the start: 6 copper layers, 63.5 x 55.9 mm, 114 parts, among them J201 JTAG Connector, J202 I2C2, J301 BWSMA-KWE-Z001, J302 BWSMA-KWE-Z001, J303 BWSMA-KWE-Z001, J501 Input Power, J502 Board1, J503 Board2, J504 Board3, J505 Board4, J601 Pipe Thermistor, J602 Ambient Thermistor, U201 CC1354P106T0RGZR, U202 LTC1694CS5TRMPBF, U401 MX25R1635FZUIL0, U501 AZ1117CH2-3.3, U502 AZ1117CH2-3.3, U602 TLV9002IDR, Y201 ABM11W-48.0000MHZ-7-B1U-T3, Y202 ABS07-32.768KHZ-T

Commit message: finished, just produce fabrication outputs
Parts:
- removed FL301, FL302, FL303: 1720BL15B0200E, 1720BL15B0200E:1720BL15B0200E
- removed J302, J303: BWSMA-KWE-Z001, digikey-footprints:RF_SMA_RightAngle_5-1814400-1
- added C301: 1pF, Capacitor_SMD:C_0402_1005Metric, F.Cu at (141.5, 128.1)
- added C302: 0.9pF, Capacitor_SMD:C_0402_1005Metric, F.Cu at (138.8, 130.2)
- added C303: 0.6pF, Capacitor_SMD:C_0402_1005Metric, F.Cu at (137.2, 132.5)
- added C304: 100pF, Capacitor_SMD:C_0402_1005Metric, F.Cu at (147.1, 130.0)
- added C305: 1pF, Capacitor_SMD:C_0402_1005Metric, F.Cu at (141.1, 126.1)
- added C306: 12pF, Capacitor_SMD:C_0402_1005Metric, F.Cu at (136.8, 133.9)
- added C307: 12pF, Capacitor_SMD:C_0402_1005Metric, F.Cu at (142.3, 128.7)
- added C308: 3pF, Capacitor_SMD:C_0402_1005Metric, F.Cu at (145.1, 127.9)
- added C309: 3pF, Capacitor_SMD:C_0402_1005Metric, F.Cu at (146.1, 129.7)
- added C310: 7pF, Capacitor_SMD:C_0402_1005Metric, F.Cu at (144.9, 133.8)
- added C311: 3.9pF, Capacitor_SMD:C_0402_1005Metric, F.Cu at (144.1, 136.5)
- added C312: 100pF, Capacitor_SMD:C_0402_1005Metric, F.Cu at (143.3, 137.7)
- added C313: 3pF, Capacitor_SMD:C_0402_1005Metric, F.Cu at (144.8, 130.8)
- added C314: 2.6pF, Capacitor_SMD:C_0402_1005Metric, F.Cu at (146.6, 126.2)
- added C315: 100pF, Capacitor_SMD:C_0402_1005Metric, F.Cu at (149.3, 130.1)
- added C316: 100pF, Capacitor_SMD:C_0402_1005Metric, F.Cu at (149.0, 129.1)
- added C317: 2.4pF, Capacitor_SMD:C_0402_1005Metric, F.Cu at (151.6, 127.4)
- added C318: 2.4pF, Capacitor_SMD:C_0402_1005Metric, F.Cu at (150.5, 129.1)
- added C319: 1.1pF, Capacitor_SMD:C_0402_1005Metric, F.Cu at (151.2, 131.8)
- added C320: 5.1pF, Capacitor_SMD:C_0402_1005Metric, F.Cu at (152.3, 135.9)
- added C321: 3.9pF, Capacitor_SMD:C_0402_1005Metric, F.Cu at (151.7, 133.2)
- added C322: 100pF, Capacitor_SMD:C_0402_1005Metric, F.Cu at (153.1, 137.1)
- added C323: 3.9pF, Capacitor_SMD:C_0402_1005Metric, F.Cu at (151.8, 130.2)
- added J304: BWSMA-KWE-Z001, digikey-footprints:RF_SMA_RightAngle_5-1814400-1, F.Cu at (133.7, 142.3)
- added J305: BWSMA-KWE-Z001, digikey-footprints:RF_SMA_RightAngle_5-1814400-1, F.Cu at (143.5, 142.3)
- added L301: 20nH, Inductor_SMD:L_0402_1005Metric, F.Cu at (142.5, 125.9)
- added L302: 3.7nH, Inductor_SMD:L_0402_1005Metric, F.Cu at (142.7, 127.3)
- added L303: 3.7nH, Inductor_SMD:L_0402_1005Metric, F.Cu at (140.7, 127.5)
- added L304: 3.4nH, Inductor_SMD:L_0402_1005Metric, F.Cu at (140.0, 129.3)
- added L305: 3.9nH, Inductor_SMD:L_0402_1005Metric, F.Cu at (138.4, 131.6)
- added L306: 10nH, Inductor_SMD:L_0402_1005Metric, F.Cu at (147.0, 128.4)
- added L307: 22nH, Inductor_SMD:L_0402_1005Metric, F.Cu at (146.3, 127.1)
- added L308: 10nH, Inductor_SMD:L_0402_1005Metric, F.Cu at (145.2, 129.4)
- added L309: 6.8nH, Inductor_SMD:L_0402_1005Metric, F.Cu at (144.8, 132.3)
- added L310: 6.8nH, Inductor_SMD:L_0402_1005Metric, F.Cu at (144.1, 135.0)
- added L311: 3.4nH, Inductor_SMD:L_0402_1005Metric, F.Cu at (147.5, 124.8)
- added L312: 3.4nH, Inductor_SMD:L_0402_1005Metric, F.Cu at (146.5, 124.6)
- added L313: 0.6nH, Inductor_SMD:L_0402_1005Metric, F.Cu at (145.0, 135.3)
- added L314: 1nH, Inductor_SMD:L_0402_1005Metric, F.Cu at (149.5, 125.4)
- added L315: 1nH, Inductor_SMD:L_0402_1005Metric, F.Cu at (150.4, 125.2)
- added L316: 12nH, Inductor_SMD:L_0402_1005Metric, F.Cu at (149.6, 127.9)
- added L317: 27nH, Inductor_SMD:L_0402_1005Metric, F.Cu at (150.4, 126.7)
- added L318: 12nH, Inductor_SMD:L_0402_1005Metric, F.Cu at (151.4, 128.9)
- added L319: 3nH, Inductor_SMD:L_0402_1005Metric, F.Cu at (152.2, 131.6)
- added L320: 5.1nH, Inductor_SMD:L_0402_1005Metric, F.Cu at (152.4, 134.4)
- added L321: 1.9nH, Inductor_SMD:L_0402_1005Metric, F.Cu at (150.2, 132.1)
- TP503: renamed from 3V3 F
- moved J301 18.4 mm to (153.1, 142.4)
- moved C202 4.16 mm to (155.5, 126.6), turned to -55 degrees
- moved C206 3.99 mm to (154.2, 127.5), turned to -55 degrees
- moved Y202 0.78 mm to (153.7, 124.5)
- renumbered UART1 to J203, UART2 to J204, UART4 to J205, UART3 to J206, PRESSURE to J603, HUMIDITY to J604, J:12V to JP501, J:5V to JP502, J:3V3 to JP503, 5V to TP501, 3V3 to TP502, Pipe to TP601, Amb to TP602
Connections:
- J301 pad 1: /RF/2.4_GHZ_SE -> /RF/PA_SE
- PS501 pad 4_1: +5V -> (no net)
- PS501 pad 4_2: +5V -> (no net)
- PS501 pad 4_3: +5V -> (no net)
- PS501 pad 4_4: +5V -> (no net)
- PS501 pad 4_5: +5V -> (no net)
- PS501 pad 4_6: +5V -> (no net)
- U201 pad 7: unconnected-(U201A-RX_TX-Pad7) -> /MCU/RF_RX_TX
Routing:
- net /MCU/RF_RX_TX: track 0.00 -> 14.7 mm, vias 0 -> 3
- net MCU_3V3_VFD: track 26.2 -> 38.8 mm, vias 13 -> 14
- net /MCU/RF_SUB_P: track 13.6 -> 3.18 mm
- net /MCU/RF_SUB_N: track 13.5 -> 3.16 mm
- net /MCU/RF_PA_N: track 12.1 -> 3.51 mm
- net /MCU/RF_PA_P: track 12.0 -> 3.55 mm
- net GND: track 58.0 -> 49.6 mm, vias 77 -> 350
- net /MCU/RF_2.4_N: track 14.9 -> 8.97 mm
- net /MCU/RF_2.4_P: track 12.9 -> 8.55 mm
- net Net-(C318-Pad2): track 0.00 -> 4.27 mm
- net Net-(C309-Pad1): track 0.00 -> 4.00 mm
- net Net-(C308-Pad2): track 0.00 -> 4.00 mm
- net Net-(C309-Pad2): track 0.00 -> 3.16 mm
- net Net-(C319-Pad2): track 0.00 -> 3.12 mm
- net Net-(C318-Pad1): track 0.00 -> 3.00 mm
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
Commit message: added mounting holes and produced manufacturing files, ALL IS DONE Alhamdulillah
Parts:
- moved J505 0.17 mm to (160.8, 142.7)
Routing:
- net GND: vias 350 -> 404
Other:
- board size 63.5 x 55.9 mm -> 63.5 x 63.1 mm
